File: kicad/room-node/audio_out.kicad_sch (KiCad schematic)
At the start: 0 parts

Commit message: SQU-27: Draw rev A schematic (6 sheets + root hierarchy)
- Draw mcu, audio_out, microphone, led_ring, sensors and display sheets
  from docs/pcb/schematic.md: doc refs, values, footprints, MPN and LCSC
  fields. The old MCU sheet (2xx refs, wiring errors) is redrawn.
- Root sheet now holds the 6 sheets as a normal hierarchy; the project
  no longer lists every file as a KiCad 10 top-level sheet, so project
  ERC and netlist cover all sheets.
- Project library: replace the wrong 4-pin AHT20 with a 6-pin symbol and
  6-pad footprint from LCSC C2757850 (pin 1 top-left, datasheet v1.1 s3);
  remove the wrong SPH0645 part (stock part is used); fix the library
  header so KiCad can load it (kicad_symbol_lib, version 20251024).
- tools/check_pinout.py: checks the netlist against pinout.md and the
  other end of each net against schematic.md.
- reports/schematic: ERC report (0 errors, 1 warning), netlist check
  (PASS), PDF of all 7 sheets.
- schematic.md: update status, refs and library notes.

Co-Authored-By: Claude Opus 5.5 <noreply@anthropic.com>
Parts:
- added C20: 470µF 16V, Capacitor_THT:CP_Radial_D8.0mm_P3.50mm, symbol Device:C_Polarized
- added C21: 0.1µF, Capacitor_SMD:C_0603_1608Metric, symbol Device:C
- added C22: 10µF 16V, Capacitor_SMD:C_0805_2012Metric, symbol Device:C
- added J2: Speaker 8Ω, Connector_JST:JST_PH_B2B-PH-SM4-TB_1x02-1MP_P2.00mm_Vertical, symbol Connector_Generic:Conn_01x02
- added R20: 100k, Resistor_SMD:R_0603_1608Metric, symbol Device:R
- added U3: MAX98357AETE+, Package_DFN_QFN:TQFN-16-1EP_3x3mm_P0.5mm_EP1.23x1.23mm, symbol Audio:MAX98357A
Connections:
- new net: J2.2 (Pin_2), U3.10 (OUTN)
- new net: J2.1 (Pin_1), U3.9 (OUTP)
- new net +5V: C20.1, C21.1, C22.1, U3.2 (GAIN_SLOT), U3.7 (VDD), U3.8 (VDD)
- new net AMP_SD: R20.1, U3.4 (~{SD_MODE})
- new net GND: C20.2, C21.2, C22.2, R20.2, U3.11 (GND), U3.15 (GND), U3.17 (PAD), U3.3 (GND)
- new net I2S_SPK_BCLK: U3.16 (BCLK)
- new net I2S_SPK_DIN: U3.1 (DIN)
- new net I2S_SPK_LRCLK: U3.14 (LRCLK)
Other:
- note added: "At U3 VDD (pins 7, 8)"
- note added: "GAIN_SLOT to VDD = 6 dB gain (tested on the breadboard; 9 dB clips). SD_MODE: R20 100k keeps the amp off during boot. GPIO HIGH = on, left channel. EP (pin 17) is not connected inside the chip: wire it to GND, vias in the pad. C20 + C21 + star ground removed the breadboard crackle. Keep all three, at the chip. Speaker: Dayton CE32A-8 (8 Ω). Do not connect either speaker wire to GND. NC pins 5, 6,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"
- note added: "I2S class-D amplifier (MAX98357A) -> speaker"
- company: (none) -> Squarewave Labs
- title: (none) -> Room node rev A - Audio out
