File: kicad/room-node/display.kicad_sch (KiCad schematic)
At the start: 0 parts

Commit message: SQU-27: Draw rev A schematic (6 sheets + root hierarchy)
- Draw mcu, audio_out, microphone, led_ring, sensors and display sheets
  from docs/pcb/schematic.md: doc refs, values, footprints, MPN and LCSC
  fields. The old MCU sheet (2xx refs, wiring errors) is redrawn.
- Root sheet now holds the 6 sheets as a normal hierarchy; the project
  no longer lists every file as a KiCad 10 top-level sheet, so project
  ERC and netlist cover all sheets.
- Project library: replace the wrong 4-pin AHT20 with a 6-pin symbol and
  6-pad footprint from LCSC C2757850 (pin 1 top-left, datasheet v1.1 s3);
  remove the wrong SPH0645 part (stock part is used); fix the library
  header so KiCad can load it (kicad_symbol_lib, version 20251024).
- tools/check_pinout.py: checks the netlist against pinout.md and the
  other end of each net against schematic.md.
- reports/schematic: ERC report (0 errors, 1 warning), netlist check
  (PASS), PDF of all 7 sheets.
- schematic.md: update status, refs and library notes.

Co-Authored-By: Claude Opus 5.5 <noreply@anthropic.com>
Parts:
- added C50: 0.1µF, Capacitor_SMD:C_0603_1608Metric, symbol Device:C
- added J3: Waveshare e-paper, Connector_JST:JST_PH_B8B-PH-SM4-TB_1x08-1MP_P2.00mm_Vertical, symbol Connector_Generic:Conn_01x08
Connections:
- new net +3V3: C50.1, J3.1 (Pin_1)
- new net EPD_BUSY: J3.8 (Pin_8)
- new net EPD_CLK: J3.4 (Pin_4)
- new net EPD_CS: J3.5 (Pin_5)
- new net EPD_DC: J3.6 (Pin_6)
- new net EPD_MOSI: J3.3 (Pin_3)
- new net EPD_RST: J3.7 (Pin_7)
- new net GND: C50.2, J3.2 (Pin_2)
Other:
- note added: "At J3 pin 1"
- note added: "BUSY"
- note added: "CLK"
- note added: "CS"
- note added: "Check the pin order and count on your cable. Newer Waveshare modules have a 9th pin (PWR): if yours has it, use a 9-pin connector and tie PWR to +3V3. Cable: needs a PH-to-PH 8-pin cable that maps pin 1 to pin 1 (beep it out before power-on). Option: 1x8 2.54 mm header (PinHeader_1x08_P2.54mm_Vertical) for the existing jumper wires. Same pin order either way."
- note added: "DC"
- note added: "DIN"
- note added: "GND"
- note added: "RST"
- note added: "VCC"
- note added: "Waveshare 2.9" e-paper module (with its driver board) via cable"
- company: (none) -> Squarewave Labs
- title: (none) -> Room node rev A - Display
