File: kicad/room-node/display.kicad_sch (KiCad schematic)
At the start: 2 parts, among them J3 Waveshare e-paper

Commit message: SQU-33: LCSC number C265121 for J3 side-entry JST S8B-PH-SM4-TB(LF)(SN)
Replaced TBD-SQU-32 with C265121 in BOM CSV and KiCad schematic.
Price at qty 10: /usr/bin/bash.3674 (Extended class, stock 19264, Active).

Co-Authored-By: Paperclip <noreply@paperclip.ing>
Parts:
- J3: footprint Connector_JST:JST_PH_B8B-PH-SM4-TB_1x08-1MP_P2.00mm_Vertical -> Connector_JST:JST_PH_S8B-PH-SM4-TB_1x08-1MP_P2.00mm_Horizontal; LCSC TBD -> C265121; MPN JST B8B-PH-SM4-TB(LF)(SN) -> JST S8B-PH-SM4-TB(LF)(SN)
Changed lines of the file:
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@@
 			)
 		)
-		(property "Footprint" "Connector_JST:JST_PH_B8B-PH-SM4-TB_1x08-1MP_P2.00mm_Vertical"
+		(property "Footprint" "Connector_JST:JST_PH_S8B-PH-SM4-TB_1x08-1MP_P2.00mm_Horizontal"
 			(at 203.2 101.6 0)
 			(hide yes)
@@
 			)
 		)
-		(property "MPN" "JST B8B-PH-SM4-TB(LF)(SN)"
+		(property "MPN" "JST S8B-PH-SM4-TB(LF)(SN)"
 			(at 203.2 101.6 0)
 			(hide yes)
@@
 			)
 		)
-		(property "LCSC" "TBD"
+		(property "LCSC" "C265121"
 			(at 203.2 101.6 0)
 			(hide yes)
