File: kicad/room-node/microphone.kicad_sch (KiCad schematic)
At the start: 0 parts

Commit message: SQU-27: Draw rev A schematic (6 sheets + root hierarchy)
- Draw mcu, audio_out, microphone, led_ring, sensors and display sheets
  from docs/pcb/schematic.md: doc refs, values, footprints, MPN and LCSC
  fields. The old MCU sheet (2xx refs, wiring errors) is redrawn.
- Root sheet now holds the 6 sheets as a normal hierarchy; the project
  no longer lists every file as a KiCad 10 top-level sheet, so project
  ERC and netlist cover all sheets.
- Project library: replace the wrong 4-pin AHT20 with a 6-pin symbol and
  6-pad footprint from LCSC C2757850 (pin 1 top-left, datasheet v1.1 s3);
  remove the wrong SPH0645 part (stock part is used); fix the library
  header so KiCad can load it (kicad_symbol_lib, version 20251024).
- tools/check_pinout.py: checks the netlist against pinout.md and the
  other end of each net against schematic.md.
- reports/schematic: ERC report (0 errors, 1 warning), netlist check
  (PASS), PDF of all 7 sheets.
- schematic.md: update status, refs and library notes.

Co-Authored-By: Claude Opus 5.5 <noreply@anthropic.com>
Parts:
- added C10: 0.1µF, Capacitor_SMD:C_0603_1608Metric, symbol Device:C
- added C11: 100pF C0G, Capacitor_SMD:C_0603_1608Metric, symbol Device:C
- added MK1: SPH0645LM4H-B, Sensor_Audio:Knowles_SPH0645LM4H-6_3.5x2.65mm, symbol Sensor_Audio:SPH0645LM4H
- added R10, R11, R9: 33Ω, Resistor_SMD:R_0603_1608Metric, symbol Device:R
- added R8: 100k, Resistor_SMD:R_0603_1608Metric, symbol Device:R
Connections:
- new net: MK1.1 (WS), R10.1
- new net: MK1.6 (DATA), R11.1
- new net: MK1.4 (BCLK), R9.1
- new net +3V3: C10.1, C11.1, MK1.5 (VDD)
- new net GND: C10.2, C11.2, MK1.2 (SEL), MK1.3 (GND), R8.2
- new net I2S_MIC_BCLK: R9.2
- new net I2S_MIC_DATA: R11.2, R8.1
- new net I2S_MIC_WS: R10.2
Other:
- note added: "At MK1 VDD (pin 5)"
- note added: "I2S MEMS microphone (SPH0645LM4H-B)"
- note added: "SELECT (pin 2) to GND = left channel. R9/R10 (33 Ω) at U1, R11 at MK1: optional damping; use 0 Ω if removed. R8 100k on I2S_MIC_DATA to GND. C11 100 pF C0G is DNP (do not fit). Use the stock symbol/footprint (Sensor_Audio). Footprint has the sound hole; GND ring around it. Mic mute is software only (no mute switch)."
- company: (none) -> Squarewave Labs
- title: (none) -> Room node rev A - Microphone
