File: kicad/room-node/room-node.kicad_sch (KiCad schematic)
At the start: 0 parts

Commit message: Decide rev A is hand-built; log Phase 2 design decisions
Rev A is assembled by hand rather than JLCPCB PCBA. Cost is close and the ~1
week lead time is tolerable; the reason is that rev A is a bring-up board for
our own house whose job is to be wrong in informative ways. Bench rework beats
assembly polish, hand-building removes any dependency on JLCPCB part stock, and
it teaches the DFM lessons the Phase 4 pilot needs. PCBA returns at the pilot.

Constrains the design: 4-layer with a solid ground plane, ENIG, stencil ordered
with the boards, single-sided placement, >=0.5mm passive spacing, 0603 minimum,
through-hole audio bulk cap, tented thermal vias, windowpaned stencil apertures
on exposed pads.

Known risk recorded: the WROOM-1 ground pad and MAX98357A thermal pad can't be
inspected once placed, and marginal joints there mimic design bugs. Bring-up
order added so assembly faults get ruled out before the schematic.

Also backfills Decisions log entries that were only living in the schematic
docs: MAX98357A kept over a PCM5102A+PAM8302A split, VA button GPIO0 -> GPIO38,
3V3 stays linear, module is N16R8. Status section refreshed for a fresh session.

Co-Authored-By: Claude Opus 5 <noreply@anthropic.com>
Other:
- title: (none) -> ${BOARD}
Changed lines of the file:
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@@
 	(generator_version "10.0")
 	(paper "A4")
+	(title_block
+		(title "${BOARD}")
+		(date "2026-07-28")
+		(rev "${REV}")
+	)
 	(sheet_instances
 		(path "/"

Commit message: SQU-27: Draw rev A schematic (6 sheets + root hierarchy)
- Draw mcu, audio_out, microphone, led_ring, sensors and display sheets
  from docs/pcb/schematic.md: doc refs, values, footprints, MPN and LCSC
  fields. The old MCU sheet (2xx refs, wiring errors) is redrawn.
- Root sheet now holds the 6 sheets as a normal hierarchy; the project
  no longer lists every file as a KiCad 10 top-level sheet, so project
  ERC and netlist cover all sheets.
- Project library: replace the wrong 4-pin AHT20 with a 6-pin symbol and
  6-pad footprint from LCSC C2757850 (pin 1 top-left, datasheet v1.1 s3);
  remove the wrong SPH0645 part (stock part is used); fix the library
  header so KiCad can load it (kicad_symbol_lib, version 20251024).
- tools/check_pinout.py: checks the netlist against pinout.md and the
  other end of each net against schematic.md.
- reports/schematic: ERC report (0 errors, 1 warning), netlist check
  (PASS), PDF of all 7 sheets.
- schematic.md: update status, refs and library notes.

Co-Authored-By: Claude Opus 5.5 <noreply@anthropic.com>
Other:
- added sheet Audio Out (audio_out.kicad_sch)
- added sheet Display (display.kicad_sch)
- added sheet LED Ring (led_ring.kicad_sch)
- added sheet MCU, Power, & USB (mcu.kicad_sch)
- added sheet Microphone (microphone.kicad_sch)
- added sheet Sensors (sensors.kicad_sch)
- note added: "Rev A room node: ESP32-S3-WROOM-1-N16R8, USB-C 5 V in, 3.3 V LDO. All sheets connect through global labels and the +5V / +3V3 / GND power symbols. Source of truth: docs/pcb/schematic.md and docs/pcb/pinout.md. Power tree: USB-C VBUS (+5V) -> AP7361C LDO -> +3V3 (module, mic, AHT20, e-paper). +5V also feeds the MAX98357A amp and the LED strip."
- company: (none) -> Squarewave Labs
- title: ${BOARD} -> Room node rev A
