File: kicad/room-node/sensors.kicad_sch (KiCad schematic)
At the start: 0 parts

Commit message: SQU-27: Draw rev A schematic (6 sheets + root hierarchy)
- Draw mcu, audio_out, microphone, led_ring, sensors and display sheets
  from docs/pcb/schematic.md: doc refs, values, footprints, MPN and LCSC
  fields. The old MCU sheet (2xx refs, wiring errors) is redrawn.
- Root sheet now holds the 6 sheets as a normal hierarchy; the project
  no longer lists every file as a KiCad 10 top-level sheet, so project
  ERC and netlist cover all sheets.
- Project library: replace the wrong 4-pin AHT20 with a 6-pin symbol and
  6-pad footprint from LCSC C2757850 (pin 1 top-left, datasheet v1.1 s3);
  remove the wrong SPH0645 part (stock part is used); fix the library
  header so KiCad can load it (kicad_symbol_lib, version 20251024).
- tools/check_pinout.py: checks the netlist against pinout.md and the
  other end of each net against schematic.md.
- reports/schematic: ERC report (0 errors, 1 warning), netlist check
  (PASS), PDF of all 7 sheets.
- schematic.md: update status, refs and library notes.

Co-Authored-By: Claude Opus 5.5 <noreply@anthropic.com>
Parts:
- added C40: 0.1µF, Capacitor_SMD:C_0603_1608Metric, symbol Device:C
- added R40, R41: 4.7k, Resistor_SMD:R_0603_1608Metric, symbol Device:R
- added U6: AHT20, room-node:AHT20, symbol room-node-lib:AHT20
Connections:
- new net +3V3: C40.1, R40.1, R41.1, U6.2 (VDD)
- new net GND: C40.2, U6.5 (GND)
- new net I2C_SCL: R41.2, U6.3 (SCL)
- new net I2C_SDA: R40.2, U6.4 (SDA)
Other:
- note added: "At U6 VDD"
- note added: "I2C pull-ups"
- note added: "Pin 1 and 6 are NC on the AHT20 (no-connect pin type). Project-library part re-made from LCSC C2757850 (6 pads, 1.0 mm pitch); pinout per Aosong AHT20 datasheet v1.1 section 3. Place U6 on a board edge, far from U1, U2, U3 and J4, with slots on three sides (board heat reads as room temperature)."
- note added: "Temperature / humidity (AHT20, I2C 0x38)"
- company: (none) -> Squarewave Labs
- title: (none) -> Room node rev A - Sensors
